File: LED_Breakout_Rev1/LED_Breakout_Rev1.kicad_sch (KiCad schematic)
At the start: 68 parts, among them Q1 PMOS, U1 74LS154, U2 74LS154

Commit message: switch voltage symbols
Parts:
- removed Conn2: Molex_SL_05, symbol MRDT_Connectors:Molex_SL_05
- removed Conn3: Molex_SL_02, symbol MRDT_Connectors:Molex_SL_02
- added U3: 74LS148, symbol 74xx:74LS148
Other:
- note removed: "5V"
- note removed: "LED_signal"
- note removed: "alternative design:"
Changed lines of the file:
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@@
     (stroke (width 0) (type default))
   )
-  (wire (pts (xy 252.73 138.43) (xy 251.46 138.43))
-    (stroke (width 0) (type default))
-  )
   (wire (pts (xy 185.42 57.15) (xy 186.69 57.15))
     (stroke (width 0) (type default))
@@
     (stroke (width 0) (type default))
   )
-  (wire (pts (xy 252.73 130.81) (xy 251.46 130.81))
-    (stroke (width 0) (type default))
-  )
   (wire (pts (xy 158.75 121.92) (xy 160.02 121.92))
     (stroke (width 0) (type default))
@@
     (stroke (width 0) (type default))
   )
-  (wire (pts (xy 252.73 133.35) (xy 251.46 133.35))
-    (stroke (width 0) (type default))
-  )
   (wire (pts (xy 54.61 135.89) (xy 62.23 135.89))
     (stroke (width 0) (type default))
@@
     (stroke (width 0) (type default))
   )
-  (wire (pts (xy 252.73 135.89) (xy 251.46 135.89))
-    (stroke (width 0) (type default))
-  )
   (wire (pts (xy 172.72 92.71) (xy 172.72 93.98))
     (stroke (width 0) (type default))
@@
     (stroke (width 0) (type default))
   )
-  (wire (pts (xy 251.46 105.41) (xy 257.81 105.41))
-    (stroke (width 0) (type default))
-  )
   (wire (pts (xy 43.18 101.6) (xy 46.99 101.6))
     (stroke (width 0) (type default))
@@
     (stroke (width 0) (type default))
   )
-  (wire (pts (xy 252.73 140.97) (xy 251.46 140.97))
-    (stroke (width 0) (type default))
-  )
   (wire (pts (xy 185.42 85.09) (xy 186.69 85.09))
     (stroke (width 0) (type default))
@@
     (stroke (width 0) (type default))
   )
-  (wire (pts (xy 251.46 107.95) (xy 257.81 107.95))
-    (stroke (width 0) (type default))
-  )
   (wire (pts (xy 99.06 135.89) (xy 102.87 135.89))
     (stroke (width 0) (type default))
@@
     (effects (font (size 2 2) (thickness 0.4) bold) (justify left bottom))
   )
-  (text "LED_signal" (at 238.76 125.73 0)
-    (effects (font (size 2 2)) (justify left bottom))
-  )
-  (text "5V" (at 242.57 95.25 0)
-    (effects (font (size 2 2)) (justify left bottom))
-  )
   (text "5-to-32 decoder" (at 158.75 29.21 0)
     (effects (font (size 2 2) (thickness 0.4) bold) (justify left bottom))
@@
     (effects (font (size 2 2) (thickness 0.4) bold) (justify left bottom))
   )
-  (text "alternative design:" (at 240.03 83.82 0)
-    (effects (font (size 2 2) (thickness 0.4) bold) (justify left bottom))
-  )
   (global_label "520nm" (shape input) (at 85.09 91.44 180) (fields_autoplaced)
     (effects (font (size 1.27 1.27)) (justify right))
@@
     )
   )
-  (global_label "LED_Signal_1" (shape output) (at 252.73 133.35 0) (fields_autoplaced)
-    (effects (font (size 1.27 1.27)) (justify left))
-    (property "Intersheetrefs" "${INTERSHEET_REFS}" (at 268.2335 133.35 0)
-      (effects (font (size 1.27 1.27)) (justify left) hide)
-    )
-  )
   (global_label "580nm" (shape input) (at 85.09 123.19 180) (fields_autoplaced)
     (effects (font (size 1.27 1.27)) (justify right))
@@
     )
   )
-  (global_label "LED_Signal_3" (shape output) (at 252.73 138.43 0) (fields_autoplaced)
-    (effects (font (size 1.27 1.27)) (justify left))
-    (property "Intersheetrefs" "${INTERSHEET_REFS}" (at 268.2335 138.43 0)
-      (effects (font (size 1.27 1.27)) (justify left) hide)
-    )
-  )
   (global_label "LED_Signal_3" (shape input) (at 158.75 54.61 180) (fields_autoplaced)
     (effects (font (size 1.27 1.27)) (justify right))
@@
     )
   )
-  (global_label "LED_Signal_2" (shape output) (at 252.73 135.89 0) (fields_autoplaced)
-    (effects (font (size 1.27 1.27)) (justify left))
-    (property "Intersheetrefs" "${INTERSHEET_REFS}" (at 268.2335 135.89 0)
-      (effects (font (size 1.27 1.27)) (justify left) hide)
-    )
-  )
-  (global_label "5V" (shape output) (at 257.81 105.41 0) (fields_autoplaced)
-    (effects (font (size 1.27 1.27)) (justify left))
-    (property "Intersheetrefs" "${INTERSHEET_REFS}" (at 263.0933 105.41 0)
-      (effects (font (size 1.27 1.27)) (justify left) hide)
-    )
-  )
   (global_label "640nm" (shape output) (at 186.69 144.78 0) (fields_autoplaced)
     (effects (font (size 1.27 1.27)) (justify left))
@@
     )
   )
-  (global_label "LED_Signal_4" (shape output) (at 252.73 140.97 0) (fields_autoplaced)
-    (effects (font (size 1.27 1.27)) (justify left))
-    (property "Intersheetrefs" "${INTERSHEET_REFS}" (at 268.2335 140.97 0)
-      (effects (font (size 1.27 1.27)) (justify left) hide)
-    )
-  )
   (global_label "5V" (shape input) (at 172.72 35.56 0) (fields_autoplaced)
     (effects (font (size 1.27 1.27)) (justify left))
@@
     )
   )
-  (global_label "LED_Signal_0" (shape output) (at 252.73 130.81 0) (fields_autoplaced)
-    (effects (font (size 1.27 1.27)) (justify left))
-    (property "Intersheetrefs" "${INTERSHEET_REFS}" (at 268.2335 130.81 0)
-      (effects (font (size 1.27 1.27)) (justify left) hide)
-    )
-  )
   (symbol (lib_id "Device:R") (at 95.25 190.5 90) (unit 1)
     (in_bom yes) (on_board yes) (dnp no) (fields_autoplaced)
@@
     )
   )
-  (symbol (lib_id "MRDT_Connectors:Molex_SL_05") (at 246.38 142.24 0) (mirror y) (unit 1)
-    (in_bom yes) (on_board yes) (dnp no) (fields_autoplaced)
-    (property "Reference" "Conn2" (at 242.57 134.62 0)
-      (effects (font (size 1.524 1.524)) (justify left))
-    )
-    (property "Value" "Molex_SL_05" (at 242.57 137.16 0)
-      (effects (font (size 1.524 1.524)) (justify left))
-    )
-    (property "Footprint" "" (at 246.38 142.24 0)
-      (effects (font (size 1.524 1.524)) hide)
-    )
-    (property "Datasheet" "" (at 246.38 142.24 0)
-      (effects (font (size 1.524 1.524)) hide)
-    )
-    (pin "1")
-    (pin "2")
-    (pin "3")
-    (pin "4")
-    (pin "5")
-    (instances
-      (project "LED_Breakout_Rev1"
-        (path "/a397e8c4-041f-4feb-bb30-d63fc1f6dda3"
-          (reference "Conn2") (unit 1)
-        )
-      )
-    )
-  )
   (symbol (lib_id "Device:R") (at 39.37 167.64 90) (unit 1)
     (in_bom yes) (on_board yes) (dnp no)
@@
     )
   )
-  (symbol (lib_id "MRDT_Connectors:Molex_SL_02") (at 246.38 104.14 180) (unit 1)
-    (in_bom yes) (on_board yes) (dnp no) (fields_autoplaced)
-    (property "Reference" "Conn3" (at 245.11 99.06 0)
-      (effects (font (size 1.524 1.524)))
-    )
-    (property "Value" "Molex_SL_02" (at 245.11 101.6 0)
-      (effects (font (size 1.524 1.524)))
-    )
-    (property "Footprint" "" (at 246.38 101.6 0)
-      (effects (font (size 1.524 1.524)) hide)
-    )
-    (property "Datasheet" "" (at 246.38 101.6 0)
-      (effects (font (size 1.524 1.524)) hide)
-    )
-    (pin "1")
-    (pin "2")
-    (instances
-      (project "LED_Breakout_Rev1"
-        (path "/a397e8c4-041f-4feb-bb30-d63fc1f6dda3"
-          (reference "Conn3") (unit 1)
-        )
-      )
-    )
-  )
   (symbol (lib_id "Device:R") (at 39.37 135.89 90) (unit 1)
     (in_bom yes) (on_board yes) (dnp no)
@@
     )
   )
-  (symbol (lib_id "power:GND") (at 257.81 107.95 0) (unit 1)
-    (in_bom yes) (on_board yes) (dnp no)
-    (property "Reference" "#PWR0101" (at 257.81 114.3 0)
-      (effects (font (size 1.27 1.27)) hide)
-    )
-    (property "Value" "GND" (at 257.937 112.3442 0)
-      (effects (font (size 1.27 1.27)))
-    )
-    (property "Footprint" "" (at 257.81 107.95 0)
-      (effects (font (size 1.27 1.27)) hide)
-    )
-    (property "Datasheet" "" (at 257.81 107.95 0)
-      (effects (font (size 1.27 1.27)) hide)
-    )
-    (pin "1")
-    (instances
-      (project "blackbox_rev1"
-        (path "/3d288c4c-9fb5-45d1-b744-b70977d4743c"
-          (reference "#PWR0101") (unit 1)
-        )
-      )
-      (project "LED_Breakout_Rev1"
-        (path "/a397e8c4-041f-4feb-bb30-d63fc1f6dda3"
-          (reference "#PWR02") (unit 1)
-        )
-      )
-      (project "Spectrometer_Rev1"
-        (path "/e46df0ef-c6ff-434c-ad57-34fad0b16f11"
-          (reference "#PWR05") (unit 1)
-        )
-      )
-    )
-  )
   (symbol (lib_id "Device:LED") (at 50.8 135.89 180) (unit 1)
     (in_bom yes) (on_board yes) (dnp no)
@@
         )
       )
+    )
+  )
+  (symbol (lib_id "74xx:74LS148") (at 212.09 66.04 0) (unit 1)
+    (in_bom yes) (on_board yes) (dnp no) (fields_autoplaced)
+    (property "Reference" "U3" (at 214.2841 48.26 0)
+      (effects (font (size 1.27 1.27)) (justify left))
+    )
+    (property "Value" "74LS148" (at 214.2841 50.8 0)
+      (effects (font (size 1.27 1.27)) (justify left))
+    )
+    (property "Footprint" "" (at 212.09 66.04 0)
+      (effects (font (size 1.27 1.27)) hide)
+    )
+    (property "Datasheet" "http://www.ti.com/lit/gpn/sn74LS148" (at 212.09 66.04 0)
+      (effects (font (size 1.27 1.27)) hide)
+    )
+    (pin "1")
+    (pin "10")
+    (pin "11")
+    (pin "12")
+    (pin "13")
+    (pin "14")
+    (pin "15")
+    (pin "16")
+    (pin "2")
+    (pin "3")
+    (pin "4")
+    (pin "5")
+    (pin "6")
+    (pin "7")
+    (pin "8")
+    (pin "9")
+    (instances
+      (project "LED_Breakout_Rev1"
+        (path "/a397e8c4-041f-4feb-bb30-d63fc1f6dda3"
+          (reference "U3") (unit 1)
+        )
+      )

Commit message: import netlist for layout
Parts:
- removed U3: 74LS148, symbol 74xx:74LS148
Changed lines of the file:
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@@
-    )
-  )
-  (symbol (lib_id "74xx:74LS148") (at 212.09 66.04 0) (unit 1)
-    (in_bom yes) (on_board yes) (dnp no) (fields_autoplaced)
-    (property "Reference" "U3" (at 214.2841 48.26 0)
-      (effects (font (size 1.27 1.27)) (justify left))
-    )
-    (property "Value" "74LS148" (at 214.2841 50.8 0)
-      (effects (font (size 1.27 1.27)) (justify left))
-    )
-    (property "Footprint" "" (at 212.09 66.04 0)
-      (effects (font (size 1.27 1.27)) hide)
-    )
-    (property "Datasheet" "http://www.ti.com/lit/gpn/sn74LS148" (at 212.09 66.04 0)
-      (effects (font (size 1.27 1.27)) hide)
-    )
-    (pin "1")
-    (pin "10")
-    (pin "11")
-    (pin "12")
-    (pin "13")
-    (pin "14")
-    (pin "15")
-    (pin "16")
-    (pin "2")
-    (pin "3")
-    (pin "4")
-    (pin "5")
-    (pin "6")
-    (pin "7")
-    (pin "8")
-    (pin "9")
-    (instances
-      (project "LED_Breakout_Rev1"
-        (path "/a397e8c4-041f-4feb-bb30-d63fc1f6dda3"
-          (reference "U3") (unit 1)
-        )
-      )
     )
   )
